Commit message: Added mesh folder. Contains all .stl files for robot_test.urdf file
Adapted original .urdf of turtlebot to our Dagu robot

File: robot_simulation/urdf/robot_test.urdf (robot description, URDF)
Before this commit: robot turtlebot3_waffle, 13 links, 12 joints
Links:
- removed link camera_depth_frame
- removed link camera_depth_optical_frame
- removed link camera_link
- removed link camera_rgb_frame
- removed link camera_rgb_optical_frame
- removed link caster_back_left_link
- removed link caster_back_right_link
- removed link wheel_left_link
- removed link wheel_right_link
- added link wheel_front_left_link, mass 2.8498940e-02; collision cylinder length=0.060 radius=0.060; visual mesh filename=package://robot_simulation/meshes/dagu_tire_left.stl scale=0.1 0.1 0.1
- added link wheel_front_right_link, mass 2.8498940e-02; collision cylinder length=0.060 radius=0.060; visual mesh filename=package://robot_simulation/meshes/dagu_tire_right.stl scale=0.1 0.1 0.1
- added link wheel_rear_left_link, mass 2.8498940e-02; collision cylinder length=0.060 radius=0.060; visual mesh filename=package://robot_simulation/meshes/dagu_tire_left.stl scale=0.1 0.1 0.1
- added link wheel_rear_right_link, mass 2.8498940e-02; collision cylinder length=0.060 radius=0.060; visual mesh filename=package://robot_simulation/meshes/dagu_tire_right.stl scale=0.1 0.1 0.1
- link base_link: mass 2.2 -> 3.0; geometry collision box size=0.230 0.120 0.070; visual mesh filename=package://robot_simulation/meshes/dagu_chassis_2.stl scale=0.1 0.1 0.1
- link base_scan: mass 0.114 -> 0.170; geometry collision cylinder length=0.060 radius=0.035; visual mesh filename=package://robot_simulation/meshes/rplidar_a1m8.stl scale=0.0001 0.0001 0.0001
Joints:
- removed joint camera_depth_joint
- removed joint camera_depth_optical_joint
- removed joint camera_joint
- removed joint camera_rgb_joint
- removed joint camera_rgb_optical_joint
- removed joint caster_back_left_joint
- removed joint caster_back_right_joint
- removed joint wheel_left_joint
- removed joint wheel_right_joint
- added joint wheel_front_left_joint: type continuous, parent base_link, child wheel_front_left_link, origin xyz=0.075 0.12 -0.035 rpy=-1.57 0 0, axis 0 0 1
- added joint wheel_front_right_joint: type continuous, parent base_link, child wheel_front_right_link, origin xyz=0.075 -0.120 -0.035 rpy=-1.57 0 0, axis 0 0 1
- added joint wheel_rear_left_joint: type continuous, parent base_link, child wheel_rear_left_link, origin xyz=-0.075 0.12 -0.035 rpy=-1.57 0 0, axis 0 0 1
- added joint wheel_rear_right_joint: type continuous, parent base_link, child wheel_rear_right_link, origin xyz=-0.075 -0.120 -0.035 rpy=-1.57 0 0, axis 0 0 1
- joint base_joint: origin xyz=0 0 0.065 rpy=0 0 0 -> xyz=0 0 0.095 rpy=0 0 0
- joint scan_joint: origin xyz=-0.064 0 0.122 rpy=0 0 0 -> xyz=-0.050 0 0.083 rpy=0 0 0
