Commit message: added wheel mass. Changed friction coeff and added friction direction for x direction (rotation)

File: robot_simulation/urdf/dagu.urdf (robot description, URDF)
Before this commit: robot turtlebot3_waffle, 8 links, 7 joints
Links:
- link wheel_front_left_link: mass 2.8498940e-02 -> 0.15
- link wheel_front_right_link: mass 2.8498940e-02 -> 0.15
- link wheel_rear_left_link: mass 2.8498940e-02 -> 0.15
- link wheel_rear_right_link: mass 2.8498940e-02 -> 0.15
